Commit message: Add files via upload

File: description/lidar.xacro (robot description, xacro)
@@ -4,5 +4,5 @@
         <parent link="chassis"/>
         <child link="laser_frame"/>
-        <origin xyz="0.3 0 0.1" rpy="0 0 0"/>    <!--0.1 0 0.175-->
+        <origin xyz="0.1 0 0.075" rpy="0 0 0"/>    <!--0.1 0 0.175-->
     </joint>
     <link name="laser_frame">

File: description/robot_core.xacro (robot description, xacro)
@@ -34,22 +34,22 @@
         <parent link = "base_link" />
         <child link = "chassis" />
-        <origin xyz = "-0.05 0 0.075" />         <!-- "0 0 0" -->
+        <origin xyz = "0 0 0.05" />         <!-- "-0.05 0 0.075" --> <!-- "0 0 0.075" -->
     </joint>
     <link name="chassis" >
         <visual>
-            <origin xyz = "0.2 0 0" />        <!--"0.2 0 0.075"-->
-            <geometry>
-                <box size="0.4 0.2 0.15" />
+            <origin xyz = "0 0 0" />        <!--"0.2 0 0"-->
+            <geometry>
+                <box size="0.4 0.2 0.1" />
             </geometry>
             <material name = "white" />
         </visual>
         <collision>
-            <origin xyz = "0.2 0 0.075" />
-            <geometry>
-                <box size="0.4 0.2 0.15" />
-            </geometry>
-        </collision>
-        <xacro:inertial_box mass="1.85" x="0.4" y="0.2" z="0.15">
-            <origin xyz = "0.2 0 0.075" rpy = "0 0 0"/>
+            <origin xyz = "0 0 0" />      <!--"0.2 0 0"-->
+            <geometry>
+                <box size="0.4 0.2 0.1" />
+            </geometry>
+        </collision>
+        <xacro:inertial_box mass="1.85" x="0.4" y="0.2" z="0.1">
+            <origin xyz = "0 0 0" rpy = "0 0 0"/>          <!--xyz = "0.2 0 0.075"-->
         </xacro:inertial_box>
     </link>
@@ -67,4 +67,5 @@
         </visual>
         <collision>
+            <origin xyz="0 0 0" rpy="-${pi/2} 0 0" />
             <geometry>
                 <cylinder radius = "0.033" length = "0.026"/>
@@ -92,4 +93,5 @@
         </visual>
         <collision>
+            <origin xyz="0 0 0" rpy="${pi/2} 0 0" />
             <geometry>
                 <cylinder radius = "0.033" length = "0.026"/>
@@ -145,5 +147,5 @@
         <parent link="art_w_left"/>
         <child link="leftiii_wheel"/>
-        <origin xyz="0.05 0 0" rpy="0 0 0" />  <!-- "0.05 0 0" -->
+        <origin xyz="0 0.05 0" rpy="0 0 0" />  <!-- "0.05 0 0" -->
         <axis xyz= "0 1 0" />             <!-- rotates around y-axis -->
         <dynamics damping="0.05" friction="0.01"/>
@@ -152,5 +154,5 @@
         <parent link="art_w_right"/>
         <child link="rightiii_wheel"/>
-        <origin xyz="0.05 0 0" rpy="0 0 0" />   <!--${pi/2}-->
+        <origin xyz="0 -0.05 0" rpy="0 0 0" />   <!--${pi/2}-->
         <axis xyz= "0 1 0"/>
         <dynamics damping="0.05" friction="0.01"/>
@@ -159,5 +161,5 @@
         <parent link="base_link"/>
         <child link="art_w_left"/>
-        <origin xyz="0.25 0.121 0" rpy = "0 0 0" />
+        <origin xyz="0.15 0.071 0" rpy = "0 0 0" />
         <limit upper="0.5236" lower="-0.5236" velocity="20" effort="10"/>
         <axis xyz= "0 0 1" />             <!-- revolutes around z-axis -->
@@ -167,5 +169,5 @@
         <parent link="base_link"/>
         <child link="art_w_right"/>
-        <origin xyz="0.25 -0.121 0" rpy = "0 0 0" />
+        <origin xyz="0.15 -0.071 0" rpy = "0 0 0" />   <!-- "0.1 -0.121 0" -->
         <limit upper="0.5236" lower="-0.5236" velocity="20" effort="10"/>
         <axis xyz= "0 0 1" />
@@ -176,5 +178,5 @@
         <parent link="base_link"/>
         <child link="left_wheel"/>
-        <origin xyz = "0 0.121 0.0" rpy = "-${pi/2} 0 0" />  <!-- "0.05 0.121 0" -->
+        <origin xyz = "-0.15 0.118 0.0" rpy = "-${pi/2} 0 0" />  <!-- "0.05 0.121 0" -->
         <axis xyz = "0 0 1" />
         <dynamics damping="0.05" friction="0.01"/>
@@ -183,5 +185,5 @@
         <parent link="base_link"/>
         <child link="right_wheel"/>
-        <origin xyz = "0 -0.121 0.0" rpy = "${pi/2} 0 0" />
+        <origin xyz = "-0.15 -0.118 0.0" rpy = "${pi/2} 0 0" />
         <axis xyz = "0 0 -1" />
         <dynamics damping="0.05" friction="0.01"/>
@@ -190,6 +192,6 @@
     <gazebo reference="leftiii_wheel">
         <material>Gazebo/Green</material>
-        <mu1>1</mu1>
-        <mu2>1</mu2>
+        <mu1>0.001</mu1>
+        <mu2>0.001</mu2>
         <kp>1000000</kp>
         <kd>0.1</kd>
@@ -198,6 +200,6 @@
     <gazebo reference="rightiii_wheel">
         <material>Gazebo/Green</material>
-        <mu1>1</mu1>
-        <mu2>1</mu2>
+        <mu1>0.001</mu1>
+        <mu2>0.001</mu2>
         <kp>1000000</kp>
         <kd>0.1</kd>
