Commit message: Add files via upload

File: description/gazebo_control.xacro (robot description, xacro)
@@ -2,11 +2,17 @@
 <robot xmlns:xacro="http://www.ros.org/wiki/xacro" >
     <gazebo>
+        <!-- Wheel information -->
         <plugin name="diff_drive" filename="libgazebo_ros_diff_drive.so">
+        <num_wheel_pairs>2</num_wheel_pairs>
         <left_joint>left_wheel_joint</left_joint>
         <right_joint>right_wheel_joint</right_joint>
-        <wheel_separation>0.34</wheel_separation>
+        <left_joint>leftiii_wheel_joint</left_joint>
+        <right_joint>rightiii_wheel_joint</right_joint>
+        <wheel_separation>0.242</wheel_separation>
         <wheel_diameter>0.1</wheel_diameter>
+        <!-- Limits -->
         <max_wheel_torque>200</max_wheel_torque>
         <max_wheel_acceleration>10.0</max_wheel_acceleration>
+        <!-- Output -->
         <odometry_frame>odom</odometry_frame>
         <robot_base_frame>base_link</robot_base_frame>

File: description/lidar.xacro (robot description, xacro)
@@ -4,5 +4,5 @@
         <parent link="chassis"/>
         <child link="laser_frame"/>
-        <origin xyz="0.1 0 0.175" rpy="0 0 0"/>
+        <origin xyz="0.3 0 0.225" rpy="0 0 0"/>    <!--0.1 0 0.175-->
     </joint>
     <link name="laser_frame">

File: description/robot.urdf.xacro (robot description, xacro)
@@ -2,5 +2,6 @@
 <robot xmlns:xacro="http://www.ros.org/wiki/xacro"  name="robot">
     <xacro:include filename="robot_core.xacro" />
-    <xacro:include filename="gazebo_control.xacro" />
+    <!-- <xacro:include filename="gazebo_control.xacro" /> -->
+    <xacro:include filename="ros2_control.xacro" />
     <xacro:include filename="lidar.xacro" />
 </robot>

File: description/robot_core.xacro (robot description, xacro)
@@ -27,25 +27,26 @@
     <link name="base_footprint">
     </link>
+    <!-- CHASSIS LINK -->
     <joint name = "chassis_joint" type = "fixed">
         <parent link = "base_link" />
         <child link = "chassis" />
-        <origin xyz = "-0.1 0 0" />
+        <origin xyz = "0 0 0" />         <!-- "-0.1 0 0" -->
     </joint>
     <link name="chassis" >
         <visual>
-            <origin xyz = "0.15 0 0.075" />
+            <origin xyz = "0.2 0 0.1" />
             <geometry>
-                <box size="0.3 0.3 0.15" />
+                <box size="0.4 0.2 0.2" />
             </geometry>
             <material name = "white" />
         </visual>
         <collision>
-            <origin xyz = "0.15 0 0.075" />
+            <origin xyz = "0.2 0 0.1" />
             <geometry>
-                <box size="0.3 0.3 0.15" />
+                <box size="0.4 0.2 0.2" />
             </geometry>
         </collision>
-        <xacro:inertial_box mass="0.5" x="0.3" y="0.3" z="0.15">
-            <origin xyz = "0.15 0 0.075" rpy = "0 0 0"/>
+        <xacro:inertial_box mass="2" x="0.4" y="0.2" z="0.2">
+            <origin xyz = "0.2 0 0.1" rpy = "0 0 0"/>
         </xacro:inertial_box>
     </link>
@@ -53,8 +54,9 @@
         <material>Gazebo/White</material>
     </gazebo>
+    <!--LEFT WHEEL JOINT-->
     <joint name = "left_wheel_joint" type = "continuous">
         <parent link = "base_link" />
         <child link = "left_wheel" />
-        <origin xyz = "0 0.17 0" rpy = "-${pi/2} 0 0" />
+        <origin xyz = "0.05 0.121 0" rpy = "-${pi/2} 0 0" />
         <axis xyz = "0 0 1" />
     </joint>
@@ -81,5 +83,5 @@
         <parent link = "base_link" />
         <child link = "leftiii_wheel" />
-        <origin xyz = "0.1 0.17 0" rpy = "-${pi/2} 0 0" />
+        <origin xyz = "0.35 0.121 0" rpy = "-${pi/2} 0 0" />
         <axis xyz = "0 0 1" />
     </joint>
@@ -89,5 +91,5 @@
                 <cylinder radius = "0.05" length = "0.04"/>
             </geometry>
-            <material name = "blue" />
+            <material name = "green" />
         </visual>
         <collision>
@@ -101,10 +103,11 @@
     </link>
     <gazebo reference="leftiii_wheel">
-        <material>Gazebo/Blue</material>
+        <material>Gazebo/Green</material>
     </gazebo>
+    <!--RIGHT WHEELS-->
     <joint name = "right_wheel_joint" type = "continuous">
         <parent link = "base_link" />
         <child link = "right_wheel" />
-        <origin xyz = "0 -0.17 0" rpy = "${pi/2} 0 0" />
+        <origin xyz = "0.05 -0.121 0" rpy = "${pi/2} 0 0" />
         <axis xyz = "0 0 -1" />
     </joint>
@@ -131,5 +134,5 @@
         <parent link = "base_link" />
         <child link = "rightiii_wheel" />
-        <origin xyz = "0.1 -0.17 0" rpy = "${pi/2} 0 0" />
+        <origin xyz = "0.35 -0.121 0" rpy = "${pi/2} 0 0" />
         <axis xyz = "0 0 -1" />
     </joint>
@@ -139,5 +142,5 @@
                 <cylinder radius = "0.05" length = "0.04"/>
             </geometry>
-            <material name = "blue" />
+            <material name = "green" />
         </visual>
         <collision>
@@ -151,7 +154,7 @@
     </link>
     <gazebo reference="rightiii_wheel">
-        <material>Gazebo/Blue</material>
+        <material>Gazebo/Green</material>
     </gazebo>
-    <joint name = "caster_wheel_joint" type = "fixed">
+    <!-- <joint name = "caster_wheel_joint" type = "fixed">
         <parent link = "chassis" />
         <child link = "caster_wheel" />
@@ -178,4 +181,4 @@
         <mu1 value = "0.001"/>
         <mu2 value = "0.001"/>
-    </gazebo>
+    </gazebo> -->
 </robot>

Commit message: Add files via upload

File: description/gazebo_control.xacro (robot description, xacro)
@@ -10,5 +10,5 @@
         <right_joint>rightiii_wheel_joint</right_joint>
         <wheel_separation>0.242</wheel_separation>
-        <wheel_diameter>0.1</wheel_diameter>
+        <wheel_diameter>0.066</wheel_diameter>
         <!-- Limits -->
         <max_wheel_torque>200</max_wheel_torque>

File: description/lidar.xacro (robot description, xacro)
@@ -4,5 +4,5 @@
         <parent link="chassis"/>
         <child link="laser_frame"/>
-        <origin xyz="0.3 0 0.225" rpy="0 0 0"/>    <!--0.1 0 0.175-->
+        <origin xyz="0.3 0 0.175" rpy="0 0 0"/>    <!--0.1 0 0.175-->
     </joint>
     <link name="laser_frame">

File: description/robot.urdf.xacro (robot description, xacro)
@@ -1,7 +1,12 @@
 <?xml version="1.0"?>
 <robot xmlns:xacro="http://www.ros.org/wiki/xacro"  name="robot">
+    <xacro:arg name="use_ros2_control" default="true" />
     <xacro:include filename="robot_core.xacro" />
-    <!-- <xacro:include filename="gazebo_control.xacro" /> -->
-    <xacro:include filename="ros2_control.xacro" />
+    <xacro:if value="$(arg use_ros2_control)">
+        <xacro:include filename="ros2_control.xacro" />
+    </xacro:if>
+    <xacro:unless value="$(arg use_ros2_control)">
+        <xacro:include filename="gazebo_control.xacro" />
+    </xacro:unless>
     <xacro:include filename="lidar.xacro" />
 </robot>

File: description/robot_core.xacro (robot description, xacro)
@@ -16,4 +16,7 @@
     <material name="red">
         <color rgba = "1 0 0 1" />
+    </material>
+    <material name="green">
+        <color rgba="0.0 1.0 0.0 1.0"/>
     </material>
     <link name="base_link" >
@@ -35,18 +38,18 @@
     <link name="chassis" >
         <visual>
-            <origin xyz = "0.2 0 0.1" />
+            <origin xyz = "0.2 0 0.075" />
             <geometry>
-                <box size="0.4 0.2 0.2" />
+                <box size="0.4 0.2 0.15" />
             </geometry>
             <material name = "white" />
         </visual>
         <collision>
-            <origin xyz = "0.2 0 0.1" />
+            <origin xyz = "0.2 0 0.075" />
             <geometry>
-                <box size="0.4 0.2 0.2" />
+                <box size="0.4 0.2 0.15" />
             </geometry>
         </collision>
-        <xacro:inertial_box mass="2" x="0.4" y="0.2" z="0.2">
-            <origin xyz = "0.2 0 0.1" rpy = "0 0 0"/>
+        <xacro:inertial_box mass="1.85" x="0.4" y="0.2" z="0.15">
+            <origin xyz = "0.2 0 0.075" rpy = "0 0 0"/>
         </xacro:inertial_box>
     </link>
@@ -64,5 +67,5 @@
         <visual>
             <geometry>
-                <cylinder radius = "0.05" length = "0.04"/>
+                <cylinder radius = "0.033" length = "0.026"/>
             </geometry>
             <material name = "blue" />
@@ -70,8 +73,8 @@
         <collision>
             <geometry>
-                <cylinder radius = "0.05" length = "0.04"/>
+                <cylinder radius = "0.033" length = "0.026"/>
             </geometry>
         </collision>
-        <xacro:inertial_cylinder mass = "0.1" radius = "0.05" length = "0.04" >
+        <xacro:inertial_cylinder mass = "0.1" radius = "0.033" length = "0.026" >
             <origin xyz = "0 0 0" rpy = "0 0 0"/>
         </xacro:inertial_cylinder>
@@ -89,5 +92,5 @@
         <visual>
             <geometry>
-                <cylinder radius = "0.05" length = "0.04"/>
+                <cylinder radius = "0.033" length = "0.026"/>
             </geometry>
             <material name = "green" />
@@ -95,8 +98,8 @@
         <collision>
             <geometry>
-                <cylinder radius = "0.05" length = "0.04"/>
+                <cylinder radius = "0.033" length = "0.026"/>
             </geometry>
         </collision>
-        <xacro:inertial_cylinder mass = "0.1" radius = "0.05" length = "0.04" >
+        <xacro:inertial_cylinder mass = "0.1" radius = "0.033" length = "0.026" >
             <origin xyz = "0 0 0" rpy = "0 0 0"/>
         </xacro:inertial_cylinder>
@@ -115,5 +118,5 @@
         <visual>
             <geometry>
-                <cylinder radius = "0.05" length = "0.04"/>
+                <cylinder radius = "0.033" length = "0.026"/>
             </geometry>
             <material name = "blue" />
@@ -121,8 +124,8 @@
         <collision>
             <geometry>
-                <cylinder radius = "0.05" length = "0.04"/>
+                <cylinder radius = "0.033" length = "0.026"/>
             </geometry>
         </collision>
-        <xacro:inertial_cylinder mass = "0.1" radius = "0.05" length = "0.04" >
+        <xacro:inertial_cylinder mass = "0.1" radius = "0.033" length = "0.026" >
             <origin xyz = "0 0 0" rpy = "0 0 0"/>
         </xacro:inertial_cylinder>
@@ -140,5 +143,5 @@
         <visual>
             <geometry>
-                <cylinder radius = "0.05" length = "0.04"/>
+                <cylinder radius = "0.033" length = "0.026"/>
             </geometry>
             <material name = "green" />
@@ -146,8 +149,8 @@
         <collision>
             <geometry>
-                <cylinder radius = "0.05" length = "0.04"/>
+                <cylinder radius = "0.033" length = "0.026"/>
             </geometry>
         </collision>
-        <xacro:inertial_cylinder mass = "0.1" radius = "0.05" length = "0.04" >
+        <xacro:inertial_cylinder mass = "0.1" radius = "0.033" length = "0.026" >
             <origin xyz = "0 0 0" rpy = "0 0 0"/>
         </xacro:inertial_cylinder>
@@ -156,29 +159,3 @@
         <material>Gazebo/Green</material>
     </gazebo>
-    <!-- <joint name = "caster_wheel_joint" type = "fixed">
-        <parent link = "chassis" />
-        <child link = "caster_wheel" />
-        <origin xyz = "0.24 0 0" />
-    </joint>
-    <link name="caster_wheel" >
-        <visual>
-            <geometry>
-                <sphere radius = "0.05" />
-            </geometry>
-            <material name = "black" />
-        </visual>
-        <collision>
-            <geometry>
-                <sphere radius = "0.05" />
-            </geometry>
-        </collision>
-        <xacro:inertial_sphere mass = "0.1" radius = "0.05" >
-            <origin xyz = "0 0 0" rpy = "0 0 0"/>
-        </xacro:inertial_sphere>
-    </link>
-    <gazebo reference="caster_wheel">
-        <material>Gazebo/Black</material>
-        <mu1 value = "0.001"/>
-        <mu2 value = "0.001"/>
-    </gazebo> -->
 </robot>
