Commit message: Add files via upload

File: description/gazebo_control.xacro (robot description, xacro)
@@ -2,5 +2,41 @@
 <robot xmlns:xacro="http://www.ros.org/wiki/xacro" >
     <gazebo>
-        <!-- Wheel information -->
+        <plugin name="gazebo_ros_ackermann_drive" filename="libgazebo_ros_ackermann_drive.so">
+            <update_rate>100.0</update_rate>
+            <!-- wheels -->
+            <front_left_joint>art_wheel_left</front_left_joint>
+            <front_right_joint>art_wheel_right</front_right_joint>
+            <rear_left_joint>left_wheel_3</rear_left_joint>
+            <rear_right_joint>right_wheel_4</rear_right_joint>
+            <left_steering_joint>base_art_w_left</left_steering_joint>
+            <right_steering_joint>base_art_w_right</right_steering_joint>
+            <!-- Max absolute steer angle for tyre in radians-->
+            <!-- Any cmd_vel angular z greater than this would be capped -->
+            <max_steer>0.5236</max_steer>
+            <!-- Max absolute steering angle of steering wheel -->
+            <max_steering_angle>7.85</max_steering_angle>
+            <!-- Max absolute linear speed in m/s -->
+            <max_speed>1.5</max_speed>
+            <!-- PID tuning -->
+            <left_steering_pid_gain>1500 0 1</left_steering_pid_gain>
+            <left_steering_i_range>0 0</left_steering_i_range>
+            <right_steering_pid_gain>1500 0 1</right_steering_pid_gain>
+            <right_steering_i_range>0 0</right_steering_i_range>
+            <linear_velocity_pid_gain>1000 0 1</linear_velocity_pid_gain>
+            <linear_velocity_i_range>0 0</linear_velocity_i_range>
+            <!--input puesto por mí-->
+            <!--<command_topic>cmd_vel</command_topic>-->
+            <!-- output -->
+            <publish_odom>true</publish_odom>
+            <publish_odom_tf>true</publish_odom_tf>
+            <publish_wheel_tf>true</publish_wheel_tf>
+            <publish_distance>true</publish_distance>
+            <odometry_frame>odom</odometry_frame>
+            <robot_base_frame>base_link</robot_base_frame>
+        </plugin>
+    </gazebo>
+</robot>
+    <!-- <gazebo>
+            Wheel information
         <plugin name="diff_drive" filename="libgazebo_ros_diff_drive.so">
         <num_wheel_pairs>2</num_wheel_pairs>
@@ -11,8 +47,8 @@
         <wheel_separation>0.242</wheel_separation>
         <wheel_diameter>0.066</wheel_diameter>
-        <!-- Limits -->
+            Limits
         <max_wheel_torque>200</max_wheel_torque>
         <max_wheel_acceleration>10.0</max_wheel_acceleration>
-        <!-- Output -->
+            Output
         <odometry_frame>odom</odometry_frame>
         <robot_base_frame>base_link</robot_base_frame>
@@ -21,4 +57,3 @@
         <publish_wheel_tf>true</publish_wheel_tf>
         </plugin>
-    </gazebo>
-</robot>
+    </gazebo> -->

File: description/lidar.xacro (robot description, xacro)
@@ -4,5 +4,5 @@
         <parent link="chassis"/>
         <child link="laser_frame"/>
-        <origin xyz="0.3 0 0.175" rpy="0 0 0"/>    <!--0.1 0 0.175-->
+        <origin xyz="0.3 0 0.1" rpy="0 0 0"/>    <!--0.1 0 0.175-->
     </joint>
     <link name="laser_frame">

File: description/robot_core.xacro (robot description, xacro)
@@ -34,9 +34,9 @@
         <parent link = "base_link" />
         <child link = "chassis" />
-        <origin xyz = "0 0 0" />         <!-- "-0.1 0 0" -->
+        <origin xyz = "-0.05 0 0.075" />         <!-- "0 0 0" -->
     </joint>
     <link name="chassis" >
         <visual>
-            <origin xyz = "0.2 0 0.075" />
+            <origin xyz = "0.2 0 0" />        <!--"0.2 0 0.075"-->
             <geometry>
                 <box size="0.4 0.2 0.15" />
@@ -57,105 +57,178 @@
         <material>Gazebo/White</material>
     </gazebo>
-    <!--LEFT WHEEL JOINT-->
-    <joint name = "left_wheel_joint" type = "continuous">
-        <parent link = "base_link" />
-        <child link = "left_wheel" />
-        <origin xyz = "0.05 0.121 0" rpy = "-${pi/2} 0 0" />
+    <!-- front_left-->
+    <link name="leftiii_wheel" >
+        <visual>
+            <origin xyz="0 0 0" rpy="-${pi/2} 0 0" />
+            <geometry>
+                <cylinder radius = "0.033" length = "0.026"/>
+            </geometry>
+            <material name = "green" />
+        </visual>
+        <collision>
+            <geometry>
+                <cylinder radius = "0.033" length = "0.026"/>
+            </geometry>
+        </collision>
+        <xacro:inertial_cylinder mass = "0.1" radius = "0.033" length = "0.026" >
+            <origin xyz = "0 0 0" rpy = "0 0 0"/>
+        </xacro:inertial_cylinder>
+    </link>
+    <link name="art_w_left">
+      <inertial>
+        <origin rpy="0 0 0" xyz="0 0 0" />
+        <mass value="1" />
+        <inertia ixx="1.0" ixy="0.0" ixz="0.0" iyy="1.0" iyz="0.0" izz="1.0" />
+      </inertial>
+    </link>
+    <!-- front_right-->
+    <link name="rightiii_wheel" >
+        <visual>
+            <origin xyz="0 0 0" rpy="${pi/2} 0 0" />
+            <geometry>
+                <cylinder radius = "0.033" length = "0.026"/>
+            </geometry>
+            <material name = "green" />
+        </visual>
+        <collision>
+            <geometry>
+                <cylinder radius = "0.033" length = "0.026"/>
+            </geometry>
+        </collision>
+        <xacro:inertial_cylinder mass = "0.1" radius = "0.033" length = "0.026" >
+            <origin xyz = "0 0 0" rpy = "0 0 0"/>
+        </xacro:inertial_cylinder>
+    </link>
+    <link name="art_w_right">
+      <inertial>
+        <origin rpy="0 0 0" xyz="0 0 0" />
+        <mass value="1" />
+        <inertia ixx="1.0" ixy="0.0" ixz="0.0" iyy="1.0" iyz="0.0" izz="1.0" />
+      </inertial>
+    </link>
+    <!-- rear_left -->
+    <link name="left_wheel" >
+        <visual>
+            <geometry>
+                <cylinder radius = "0.033" length = "0.026"/>
+            </geometry>
+            <material name = "blue" />
+        </visual>
+        <collision>
+            <geometry>
+                <cylinder radius = "0.033" length = "0.026"/>
+            </geometry>
+        </collision>
+        <xacro:inertial_cylinder mass = "0.1" radius = "0.033" length = "0.026" >
+            <origin xyz = "0 0 0" rpy = "0 0 0"/>
+        </xacro:inertial_cylinder>
+    </link>
+    <!-- rear_right -->
+    <link name="right_wheel" >
+        <visual>
+            <geometry>
+                <cylinder radius = "0.033" length = "0.026"/>
+            </geometry>
+            <material name = "blue" />
+        </visual>
+        <collision>
+            <geometry>
+                <cylinder radius = "0.033" length = "0.026"/>
+            </geometry>
+        </collision>
+        <xacro:inertial_cylinder mass = "0.1" radius = "0.033" length = "0.026" >
+            <origin xyz = "0 0 0" rpy = "0 0 0"/>
+        </xacro:inertial_cylinder>
+    </link>
+<!-- //////////////////////////////// ACKERMANN STEERING JOINTS //////////////////////////////////// -->
+    <joint name="art_wheel_left" type="continuous">
+        <parent link="art_w_left"/>
+        <child link="leftiii_wheel"/>
+        <origin xyz="0.05 0 0" rpy="0 0 0" />  <!-- "0.05 0 0" -->
+        <axis xyz= "0 1 0" />             <!-- rotates around y-axis -->
+        <dynamics damping="0.05" friction="0.01"/>
+    </joint>
+    <joint name="art_wheel_right" type="continuous">
+        <parent link="art_w_right"/>
+        <child link="rightiii_wheel"/>
+        <origin xyz="0.05 0 0" rpy="0 0 0" />   <!--${pi/2}-->
+        <axis xyz= "0 1 0"/>
+        <dynamics damping="0.05" friction="0.01"/>
+    </joint>
+    <joint name="base_art_w_left" type="revolute">
+        <parent link="base_link"/>
+        <child link="art_w_left"/>
+        <origin xyz="0.25 0.121 0" rpy = "0 0 0" />
+        <limit upper="0.5236" lower="-0.5236" velocity="20" effort="10"/>
+        <axis xyz= "0 0 1" />             <!-- revolutes around z-axis -->
+        <dynamics damping="0.05" friction="0.2"/>
+    </joint>
+    <joint name="base_art_w_right" type="revolute">
+        <parent link="base_link"/>
+        <child link="art_w_right"/>
+        <origin xyz="0.25 -0.121 0" rpy = "0 0 0" />
+        <limit upper="0.5236" lower="-0.5236" velocity="20" effort="10"/>
+        <axis xyz= "0 0 1" />
+        <dynamics damping="0.05" friction="0.2"/>
+    </joint>
+<!-- ////////////////////////////////////// JOINTS ///////////////////////////////////////////////// -->
+    <joint name="left_wheel_3" type="continuous">
+        <parent link="base_link"/>
+        <child link="left_wheel"/>
+        <origin xyz = "0 0.121 0.0" rpy = "-${pi/2} 0 0" />  <!-- "0.05 0.121 0" -->
         <axis xyz = "0 0 1" />
-    </joint>
-    <link name="left_wheel" >
-        <visual>
-            <geometry>
-                <cylinder radius = "0.033" length = "0.026"/>
-            </geometry>
-            <material name = "blue" />
-        </visual>
-        <collision>
-            <geometry>
-                <cylinder radius = "0.033" length = "0.026"/>
-            </geometry>
-        </collision>
-        <xacro:inertial_cylinder mass = "0.1" radius = "0.033" length = "0.026" >
-            <origin xyz = "0 0 0" rpy = "0 0 0"/>
-        </xacro:inertial_cylinder>
-    </link>
+        <dynamics damping="0.05" friction="0.01"/>
+    </joint>
+    <joint name="right_wheel_4" type="continuous">
+        <parent link="base_link"/>
+        <child link="right_wheel"/>
+        <origin xyz = "0 -0.121 0.0" rpy = "${pi/2} 0 0" />
+        <axis xyz = "0 0 -1" />
+        <dynamics damping="0.05" friction="0.01"/>
+    </joint>
+<!-- ////////////////////////////////////// GAZEBO ///////////////////////////////////////////////// -->
+    <gazebo reference="leftiii_wheel">
+        <material>Gazebo/Green</material>
+        <mu1>1</mu1>
+        <mu2>1</mu2>
+        <kp>1000000</kp>
+        <kd>0.1</kd>
+        <selfCollide>true</selfCollide>
+    </gazebo>
+    <gazebo reference="rightiii_wheel">
+        <material>Gazebo/Green</material>
+        <mu1>1</mu1>
+        <mu2>1</mu2>
+        <kp>1000000</kp>
+        <kd>0.1</kd>
+        <selfCollide>true</selfCollide>
+    </gazebo>
     <gazebo reference="left_wheel">
         <material>Gazebo/Blue</material>
-    </gazebo>
-    <joint name = "leftiii_wheel_joint" type = "continuous">
-        <parent link = "base_link" />
-        <child link = "leftiii_wheel" />
-        <origin xyz = "0.35 0.121 0" rpy = "-${pi/2} 0 0" />
-        <axis xyz = "0 0 1" />
-    </joint>
-    <link name="leftiii_wheel" >
-        <visual>
-            <geometry>
-                <cylinder radius = "0.033" length = "0.026"/>
-            </geometry>
-            <material name = "green" />
-        </visual>
-        <collision>
-            <geometry>
-                <cylinder radius = "0.033" length = "0.026"/>
-            </geometry>
-        </collision>
-        <xacro:inertial_cylinder mass = "0.1" radius = "0.033" length = "0.026" >
-            <origin xyz = "0 0 0" rpy = "0 0 0"/>
-        </xacro:inertial_cylinder>
-    </link>
-    <gazebo reference="leftiii_wheel">
-        <material>Gazebo/Green</material>
-    </gazebo>
-    <!--RIGHT WHEELS-->
-    <joint name = "right_wheel_joint" type = "continuous">
-        <parent link = "base_link" />
-        <child link = "right_wheel" />
-        <origin xyz = "0.05 -0.121 0" rpy = "${pi/2} 0 0" />
-        <axis xyz = "0 0 -1" />
-    </joint>
-    <link name="right_wheel" >
-        <visual>
-            <geometry>
-                <cylinder radius = "0.033" length = "0.026"/>
-            </geometry>
-            <material name = "blue" />
-        </visual>
-        <collision>
-            <geometry>
-                <cylinder radius = "0.033" length = "0.026"/>
-            </geometry>
-        </collision>
-        <xacro:inertial_cylinder mass = "0.1" radius = "0.033" length = "0.026" >
-            <origin xyz = "0 0 0" rpy = "0 0 0"/>
-        </xacro:inertial_cylinder>
-    </link>
+        <mu1>1</mu1>
+        <mu2>1</mu2>
+        <kp>1000000</kp>
+        <kd>0.1</kd>
+        <selfCollide>true</selfCollide>
+    </gazebo>
     <gazebo reference="right_wheel">
         <material>Gazebo/Blue</material>
-    </gazebo>
-    <joint name = "rightiii_wheel_joint" type = "continuous">
-        <parent link = "base_link" />
-        <child link = "rightiii_wheel" />
-        <origin xyz = "0.35 -0.121 0" rpy = "${pi/2} 0 0" />
-        <axis xyz = "0 0 -1" />
-    </joint>
-    <link name="rightiii_wheel" >
-        <visual>
-            <geometry>
-                <cylinder radius = "0.033" length = "0.026"/>
-            </geometry>
-            <material name = "green" />
-        </visual>
-        <collision>
-            <geometry>
-                <cylinder radius = "0.033" length = "0.026"/>
-            </geometry>
-        </collision>
-        <xacro:inertial_cylinder mass = "0.1" radius = "0.033" length = "0.026" >
-            <origin xyz = "0 0 0" rpy = "0 0 0"/>
-        </xacro:inertial_cylinder>
-    </link>
-    <gazebo reference="rightiii_wheel">
-        <material>Gazebo/Green</material>
+        <mu1>1</mu1>
+        <mu2>1</mu2>
+        <kp>1000000</kp>
+        <kd>0.1</kd>
+        <selfCollide>true</selfCollide>
+    </gazebo>
+    <gazebo reference="art_w_left">
+      <material>Gazebo/Green</material>
+      <mu1>0.2</mu1>
+      <mu2>0.2</mu2>
+      <selfCollide>true</selfCollide>
+    </gazebo>
+    <gazebo reference="art_w_right">
+      <material>Gazebo/Green</material>
+      <mu1>0.2</mu1>
+      <mu2>0.2</mu2>
+      <selfCollide>true</selfCollide>
     </gazebo>
 </robot>

File: description/ros2_control.xacro (robot description, xacro)
@@ -21,5 +21,5 @@
             <state_interface name="position"/>
         </joint>
-        <joint name="leftiii_wheel_joint">
+        <joint name="left_steer_joint">
             <command_interface name="position">
                 <param name="min">-1.57</param>
@@ -27,6 +27,7 @@
             </command_interface>
             <state_interface name="position"/>
+            <state_interface name="velocity"/>
         </joint>
-        <joint name="rightiii_wheel_joint">
+        <joint name="right_steer_joint">
             <command_interface name="position">
                 <param name="min">-1.57</param>
@@ -34,4 +35,5 @@
             </command_interface>
             <state_interface name="position"/>
+            <state_interface name="velocity"/>
         </joint>
     </ros2_control>
@@ -42,2 +44,40 @@
     </gazebo>
 </robot>
+    <!-- <plugin name="gazebo_ros_ackermann_drive" filename="libgazebo_ros_ackermann_drive.so"> </plugin> -->
+    <!-- <ros2_control name="ackermann_ros2_control" type="system">
+        <hardware>
+            <plugin>ackermann_steering_controller/AckermannSteeringController</plugin>
+        </hardware>
+        <joint name="left_wheel_joint">
+            <command_interface name="velocity">
+                <param name="min">-10</param>
+                <param name="max">10</param>
+            </command_interface>
+            <state_interface name="velocity"/>
+            <state_interface name="position"/>
+        </joint>
+        <joint name="right_wheel_joint">
+            <command_interface name="velocity">
+                <param name="min">-10</param>
+                <param name="max">10</param>
+            </command_interface>
+            <state_interface name="velocity"/>
+            <state_interface name="position"/>
+        </joint>
+        <joint name="leftiii_wheel_joint">
+            <command_interface name="position">
+                <param name="min">-1.57</param>
+                <param name="max">1.57</param>
+            </command_interface>
+            <state_interface name="velocity"/>
+            <state_interface name="position"/>
+        </joint>
+        <joint name="rightiii_wheel_joint">
+            <command_interface name="position">
+                <param name="min">-1.57</param>
+                <param name="max">1.57</param>
+            </command_interface>
+            <state_interface name="velocity"/>
+            <state_interface name="position"/>
+        </joint>
+    </ros2_control> -->

Commit message: Add files via upload

File: description/gazebo_control.xacro (robot description, xacro)
@@ -19,12 +19,12 @@
             <max_speed>1.5</max_speed>
             <!-- PID tuning -->
-            <left_steering_pid_gain>1500 0 1</left_steering_pid_gain>
+            <left_steering_pid_gain>100 0 1</left_steering_pid_gain> <!-- 1500 0 1 -->
             <left_steering_i_range>0 0</left_steering_i_range>
-            <right_steering_pid_gain>1500 0 1</right_steering_pid_gain>
+            <right_steering_pid_gain>100 0 1</right_steering_pid_gain> <!-- 1500 0 1 -->
             <right_steering_i_range>0 0</right_steering_i_range>
-            <linear_velocity_pid_gain>1000 0 1</linear_velocity_pid_gain>
+            <linear_velocity_pid_gain>100 0 1</linear_velocity_pid_gain> <!-- 1000 0 1 -->
             <linear_velocity_i_range>0 0</linear_velocity_i_range>
             <!--input puesto por mí-->
-            <!--<command_topic>cmd_vel</command_topic>-->
+            <command_topic>cmd_vel</command_topic>
             <!-- output -->
             <publish_odom>true</publish_odom>

File: description/robot_core.xacro (robot description, xacro)
@@ -75,10 +75,15 @@
             <origin xyz = "0 0 0" rpy = "0 0 0"/>
         </xacro:inertial_cylinder>
+        <inertial>
+            <origin rpy="0 0 0" xyz="0 0 0" />
+            <mass value="0.01" />
+            <inertia ixx="10" ixy="0.0" ixz="0.0" iyy="10" iyz="0.0" izz="10" />
+        </inertial>
     </link>
     <link name="art_w_left">
       <inertial>
         <origin rpy="0 0 0" xyz="0 0 0" />
-        <mass value="1" />
-        <inertia ixx="1.0" ixy="0.0" ixz="0.0" iyy="1.0" iyz="0.0" izz="1.0" />
+        <mass value="0.01" />
+        <inertia ixx="10" ixy="0.0" ixz="0.0" iyy="10" iyz="0.0" izz="10" />
       </inertial>
     </link>
@@ -101,10 +106,15 @@
             <origin xyz = "0 0 0" rpy = "0 0 0"/>
         </xacro:inertial_cylinder>
+        <inertial>
+            <origin rpy="0 0 0" xyz="0 0 0" />
+            <mass value="0.01" />
+            <inertia ixx="10" ixy="0.0" ixz="0.0" iyy="10" iyz="0.0" izz="10" />
+        </inertial>
     </link>
     <link name="art_w_right">
       <inertial>
         <origin rpy="0 0 0" xyz="0 0 0" />
-        <mass value="1" />
-        <inertia ixx="1.0" ixy="0.0" ixz="0.0" iyy="1.0" iyz="0.0" izz="1.0" />
+        <mass value="0.01" />
+        <inertia ixx="10" ixy="0.0" ixz="0.0" iyy="10" iyz="0.0" izz="10" />
       </inertial>
     </link>
@@ -125,4 +135,9 @@
             <origin xyz = "0 0 0" rpy = "0 0 0"/>
         </xacro:inertial_cylinder>
+        <inertial>
+            <origin rpy="0 0 0" xyz="0 0 0" />
+            <mass value="0.01" />
+            <inertia ixx="10" ixy="0.0" ixz="0.0" iyy="10" iyz="0.0" izz="10" />
+        </inertial>
     </link>
     <!-- rear_right -->
@@ -142,4 +157,9 @@
             <origin xyz = "0 0 0" rpy = "0 0 0"/>
         </xacro:inertial_cylinder>
+        <inertial>
+            <origin rpy="0 0 0" xyz="0 0 0" />
+            <mass value="0.01" />
+            <inertia ixx="10" ixy="0.0" ixz="0.0" iyy="10" iyz="0.0" izz="10" />
+        </inertial>
     </link>
 <!-- //////////////////////////////// ACKERMANN STEERING JOINTS //////////////////////////////////// -->
